Commit message: Train V5.9 with corrected mechanics and USB jitter

File: model/纯底盘_v5/urdf/robot.urdf (robot description, URDF)
Before this commit: robot v5_gas_spring_closedchain_research, 19 links, 18 joints
Joints:
- joint L_joint2: limit lower=-0.17342741539177786 upper=0.6119707480056704 effort=100 velocity=100 -> lower=-0.08616095279206137 upper=1.1355695236039693 effort=100 velocity=100
- joint L_spring_slide: limit lower=-0.005470234560387616 upper=0.07452976551411819 effort=1000 velocity=100 -> lower=-0.010272819908874534 upper=0.06972718009112547 effort=1000 velocity=100
- joint R_jonit2: limit lower=-0.6119707480056704 upper=0.17342741539177786 effort=100 velocity=100 -> lower=-1.1355695236039693 upper=0.08616095279206137 effort=100 velocity=100
- joint R_spring_slide: limit lower=-0.005470234560387616 upper=0.07452976551411819 effort=1000 velocity=100 -> lower=-0.010272819908874534 upper=0.06972718009112547 effort=1000 velocity=100
